File: hw/pandore/pandore.kicad_pcb (KiCad board)
At the start: 4 copper layers, 260 x 110 mm, 412 parts, among them J1 HDMI, J10 MIDI_in, J11 MIDI_out, J12 TRS, J13 NGFF_M.2_M, J15 AIO, J16 DIO, J17 GROVE, J18 GROVE, J19 NGFF_M.2_AE, J2 USB2-A_2stacked, J3 USB3-A_2stacked, J4 XLR+TRS6.35+3SW, J5 XLR+TRS6.35+3SW, J6 VIN, J7 TRS, J8 8p8c_2led_shield, J9 8p8c_2led_shield, Q1 MOSFET_EN-N, Q2 MOSFET_EN-N, Q3 MOSFET_EN-N, Q4 MOSFET_EN-N, T1 tran_choke_center, T10 tran_choke_center, T11 tran_choke_center, T12 tran_choke_center, T13 tran_choke_center, T14 tran_choke_center, T15 tran_choke_center, T16 tran_choke_center, T2 tran_choke_center, T3 tran_choke_center, T4 tran_choke_center, T5 tran_choke_center, T6 tran_choke_center, T7 tran_choke_center, T8 tran_choke_center, T9 tran_choke_center, U1 LattePanda_Mu, U10 H11L1, U11 CS4272, U12 NXES2, U13 -, U14 -, U15 OPAMP_DIFF_1, U16 OPAMP_DIFF_1, U17 OPAMP_DIFF_1, U18 OPAMP_DIFF_1, U2 mem_flash_spi, U3 RP2350B, U4 RP2350B, U5 mem_flash_spi, U6 mem_flash_spi, U7 RTL8111H, U8 RTL8111H, U9 Teensy 4.1, X1 12MHz, 30ppm+30ppm, 10pF, X2 12MHz, 30ppm+30ppm, 10pF, X3 25MHz, 30ppm+30ppm, 10pF, X4 25MHz, 30ppm+30ppm, 10pF, X5 24.576MHz, 50ppm+20ppm, 18pF

Commit message: added power stuff revised M.2 for higher model and added m.2 mounts added power tap terminals
Parts:
- added C179: 100nF, 16V, X7R, reekilib_cap:CAPC1005, F.Cu at (242.9, 67.8)
- added C180: 22µF, 25V, X5R, reekilib_cap:CAPC3216, F.Cu at (240.7, 74.8)
- added C181: 22µF, 25V, X5R, reekilib_cap:CAPC3216, F.Cu at (240.7, 72.5)
- added C182: 22µF, 25V, X5R, reekilib_cap:CAPC3216, F.Cu at (240.7, 77.0)
- added C183: 1nF, 16V, X7R, reekilib_cap:CAPC1005, F.Cu at (244.7, 65.3)
- added C184: 68pF, 10V, X7R, reekilib_cap:CAPC1005, F.Cu at (244.7, 66.3)
- added C185: 47pF, 10V, X7R, reekilib_cap:CAPC1005, F.Cu at (249.1, 66.0)
- added C186: 10µF, 25V, X5R, reekilib_cap:CAPC2012, F.Cu at (248.4, 69.8)
- added C187: 100µF, 25V, 20%, reekilib_cap:CAPAE630Xxxx, F.Cu at (267.3, 61.2)
- added C188: 10µF, 25V, X5R, reekilib_cap:CAPC2012, F.Cu at (261.5, 70.0)
- added C189: 100nF, 16V, X7R, reekilib_cap:CAPC1005, F.Cu at (256.0, 68.2)
- added C190: 1nF, 16V, X7R, reekilib_cap:CAPC1005, F.Cu at (257.8, 65.5)
- added C191: 68pF, 10V, X7R, reekilib_cap:CAPC1005, F.Cu at (257.7, 66.5)
- added C192: 22µF, 25V, X5R, reekilib_cap:CAPC3216, F.Cu at (253.8, 77.8)
- added C193: 22µF, 25V, X5R, reekilib_cap:CAPC3216, F.Cu at (253.8, 75.5)
- added C194: 22µF, 25V, X5R, reekilib_cap:CAPC3216, F.Cu at (253.8, 73.2)
- added C195: 47pF, 10V, X7R, reekilib_cap:CAPC1005, F.Cu at (261.8, 66.2)
- added D23: green, reekilib_led:LEDM1608X80, F.Cu at (245.2, 81.2)
- added D24: green, reekilib_led:LEDM1608X80, F.Cu at (259.1, 81.5)
- added J14: VIN, reekilib_con:Wurth_691137710002, F.Cu at (275.5, 61.0)
- added J20: V5, reekilib_con:Wurth_691137710002, B.Cu at (265.8, 76.0)
- added J21: V3.3, reekilib_con:Wurth_691137710002, B.Cu at (265.8, 87.5)
- added J22: V12ISO, reekilib_con:Wurth_691137710002, F.Cu at (26.0, 103.2)
- added J23: AV5, reekilib_con:Wurth_691137710002, F.Cu at (26.0, 92.0)
- added J24: AV3P3, reekilib_con:Wurth_691137710002, F.Cu at (26.0, 80.8)
- added L4: 8.2µH, 5A, reekilib_ind:Eaton_HPAL1V0630, F.Cu at (246.7, 75.3)
- added L5: 8.2µH, 5A, reekilib_ind:Eaton_HPAL1V0630, F.Cu at (259.8, 75.5)
- added M2AE30: M2, reekilib_mnt:mnt_M2_ele, B.Cu at (171.7, 103.9)
- added M2M110: M2, reekilib_mnt:mnt_M2_ele, B.Cu at (265.4, 131.9)
- added M2M42: M2, reekilib_mnt:mnt_M2_ele, B.Cu at (197.4, 131.9)
- added M2M60: M2, reekilib_mnt:mnt_M2_ele, B.Cu at (215.4, 131.9)
- added M2M80: M2, reekilib_mnt:mnt_M2_ele, B.Cu at (235.4, 131.9)
- added Q5: MOSFET_EN-N, reekilib_sot:SOT95P280X100-3, F.Cu at (246.8, 83.8)
- added Q6: MOSFET_EN-N, reekilib_sot:SOT95P280X100-3, F.Cu at (260.3, 83.8)
- added R126: 158kΩ, 1%, 63mW, reekilib_res:RESC1005, F.Cu at (249.3, 67.0)
- added R127: 30kΩ, 1%, 63mW, reekilib_res:RESC1005, F.Cu at (247.7, 67.0)
- added R128: 68.1kΩ, 1%, 63mW, reekilib_res:RESC1005, F.Cu at (246.2, 65.8)
- added R129: 10kΩ, 1%, 63mW, reekilib_res:RESC1005, F.Cu at (247.7, 68.3)
- added R130: 10kΩ, 1%, 63mW, reekilib_res:RESC1005, F.Cu at (249.2, 68.3)
- added R131: 0Ω, 5%, thin film, reekilib_res:RESC2012, F.Cu at (242.0, 80.0)
- added R132: 1kΩ, 1%, 63mW, reekilib_res:RESC1005, F.Cu at (247.5, 81.5)
- added R133: 10kΩ, 1%, 63mW, reekilib_res:RESC1005, F.Cu at (260.6, 68.5)
- added R134: 10kΩ, 1%, 63mW, reekilib_res:RESC1005, F.Cu at (262.2, 68.5)
- added R135: 100kΩ, 1%, 63mW, reekilib_res:RESC1005, F.Cu at (259.2, 66.0)
- added R136: 93.1kΩ, 1%, 63mW, reekilib_res:RESC1005, F.Cu at (262.0, 67.2)
- added R137: 30kΩ, 1%, 63mW, reekilib_res:RESC1005, F.Cu at (260.5, 67.2)
- added R138: 0Ω, 5%, thin film, reekilib_res:RESC2012, F.Cu at (255.2, 80.5)
- added R139: 1kΩ, 1%, 63mW, reekilib_res:RESC1005, F.Cu at (261.3, 81.5)
- added R140: 10kΩ, 1%, 63mW, reekilib_res:RESC1005, F.Cu at (258.1, 84.2)
- added R141: 10kΩ, 1%, 63mW, reekilib_res:RESC1005, F.Cu at (244.5, 84.2)
- added R142: 0Ω, 5%, thin film, reekilib_res:RESC2012, F.Cu at (90.5, 106.5)
- added U19: AP6335xQ, reekilib_dfn:DFN300X200X90-9, F.Cu at (245.1, 68.9)
- added U20: AP6335xQ, reekilib_dfn:DFN300X200X90-9, F.Cu at (258.1, 69.0)
- moved V11 109.2 mm to (117.0, 144.8)
- moved V2 50.1 mm to (262.5, 141.9)
- moved V3 49.7 mm to (267.8, 142.3)
- moved R19 43.2 mm to (190.4, 92.9), turned to 180 degrees
- moved R17 41.9 mm to (190.4, 91.9), turned to 180 degrees
- moved C45 40.8 mm to (192.8, 90.1), turned to -90 degrees
- moved C46 40.3 mm to (192.0, 90.1), turned to -90 degrees
- moved C42 39.8 mm to (195.4, 87.9), turned to 0 degrees
- moved C65 39.8 mm to (188.0, 91.1), turned to 0 degrees
- moved C53 38.9 mm to (190.4, 89.7), turned to 90 degrees
- moved V1 38.9 mm to (264.6, 146.2)
- moved C41 38.8 mm to (195.4, 87.1), turned to 0 degrees
- moved C69 38.5 mm to (189.6, 89.7), turned to 90 degrees
- moved C63 38.4 mm to (188.0, 90.1), turned to 0 degrees
- moved C74 37.9 mm to (185.1, 90.4), turned to 180 degrees
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Connections:
- net /Computer/MIDI.RX renamed /Computer/AUDIO.MIDI.RX
- net /Computer/MIDI.TX renamed /Computer/AUDIO.MIDI.TX
- C103 pad 2: AV3P3 -> Net-(U14-OUT)
- C114 pad 2: AV3P3 -> Net-(U14-OUT)
- J6 pad 2: unconnected-(J6-RING-Pad2) -> VSS
- J6 pad S: unconnected-(J6-SHD-PadS) -> VSS
- R72 pad 1: AV3P3 -> Net-(U14-OUT)
- U1 pad 160: unconnected-(U1A-I2S_MCLK-Pad160) -> /Audio/CPU.MCLK
- U1 pad 162: unconnected-(U1A-I2S_SCLK-Pad162) -> /Audio/CPU.TXCLK
- U1 pad 164: unconnected-(U1A-I2S_SFRM-Pad164) -> /Audio/CPU.TXFS
- U1 pad 166: unconnected-(U1A-I2S_TXD-Pad166) -> /Audio/CPU.TXD0
- U1 pad 168: unconnected-(U1A-I2S_RXD-Pad168) -> /Audio/CPU.RXD0
- U14 pad 1: AV3P3 -> Net-(U14-OUT)

Commit message: Lots of routing done power blocks intra-routing mostly done rp2350 routing mostly done some label cleanup
Parts:
- added C196: 10µF, 25V, X5R, reekilib_cap:CAPC2012, F.Cu at (97.8, 111.2)
- added C197: 10µF, 25V, X5R, reekilib_cap:CAPC2012, F.Cu at (99.5, 111.2)
- added C198: 10µF, 25V, X5R, reekilib_cap:CAPC2012, F.Cu at (101.2, 111.2)
- added C199: 10nF, 100V, X7R, reekilib_cap:CAPC1005, F.Cu at (92.2, 98.0)
- added C200: 100nF, 25V, X7R, reekilib_cap:CAPC1005, F.Cu at (101.0, 104.0)
- added C201: 1µF, 16V, X7R, reekilib_cap:CAPC1608, F.Cu at (101.2, 105.5)
- added C202: 12nF, 16V, X7R, reekilib_cap:CAPC1005, F.Cu at (94.0, 105.5)
- added C203: 1pF, 16V, X7R, reekilib_cap:CAPC1005, F.Cu at (97.0, 102.0)
- added C204: 1nF, 16V, X7R, reekilib_cap:CAPC1005, F.Cu at (93.5, 102.0)
- added C205: 100nF, 100V, X7R, reekilib_cap:CAPC2012, F.Cu at (103.2, 109.2)
- added C206: 56µF, 100V, 20%, reekilib_cap:CAPAE1000Xxxx, F.Cu at (108.2, 101.8)
- added C207: 10µF, 100V, X5R, reekilib_cap:CAPC3225, F.Cu at (106.8, 109.0)
- added C208: 56µF, 100V, 20%, reekilib_cap:CAPAE1000Xxxx, F.Cu at (85.5, 100.8)
- added C209: 100nF, 100V, X7R, reekilib_cap:CAPC2012, F.Cu at (96.0, 95.8)
- added C210: 100pF, 1kV, X5R, reekilib_cap:CAPC3216, F.Cu at (124.0, 106.8)
- added C211: 100pF, 1kV, X5R, reekilib_cap:CAPC3216, B.Cu at (124.0, 106.8)
- added C212: 100pF, 1kV, X5R, reekilib_cap:CAPC3216, F.Cu at (128.0, 54.3)
- added C213: 100pF, 1kV, X5R, reekilib_cap:CAPC3216, B.Cu at (128.0, 54.2)
- added C214: 4.7µF, 6.3V, X5R, reekilib_cap:CAPC1005, F.Cu at (242.2, 94.2)
- added C215: 4.7µF, 6.3V, X5R, reekilib_cap:CAPC1005, F.Cu at (266.3, 116.6)
- added C216: 4.7µF, 6.3V, X5R, reekilib_cap:CAPC1005, F.Cu at (242.2, 97.0)
- added C217: 4.7µF, 6.3V, X5R, reekilib_cap:CAPC1005, F.Cu at (264.4, 114.6)
- added C218: 4.7µF, 6.3V, X5R, reekilib_cap:CAPC1005, F.Cu at (239.8, 96.5)
- added C219: 4.7µF, 6.3V, X5R, reekilib_cap:CAPC1005, F.Cu at (266.4, 113.3)
- added D25: 100V, 150mA, 450mV@10mA, reekilib_sod:sod-123, F.Cu at (99.5, 108.0)
- added D26: green, reekilib_led:LEDM1608X80, F.Cu at (95.8, 90.5)
- added J26: PPWR, reekilib_con:HDR254P1X02-TH, F.Cu at (68.8, 82.0)
- added JMP3: PPWR, reekilib_con:HDR254P1X02-TH, F.Cu at (97.2, 82.2)
- added L6: Ind, reekilib_ind:WE_IND5030, F.Cu at (93.8, 110.0)
- added L7: 3.3µH, 1.8A, reekilib_ind:INDC2012, F.Cu at (241.8, 95.6)
- added L8: 3.3µH, 1.8A, reekilib_ind:INDC2012, F.Cu at (265.6, 115.3)
- added Q7: MOSFET_EN-N, reekilib_sot:SOT95P280X100-3, F.Cu at (97.2, 92.7)
- added R143: 10kΩ, 1%, 63mW, reekilib_res:RESC1005, F.Cu at (100.7, 97.7)
- added R144: 10kΩ, 1%, 63mW, reekilib_res:RESC1005, F.Cu at (100.7, 99.2)
- added R145: 10kΩ, 1%, 63mW, reekilib_res:RESC1005, F.Cu at (93.2, 97.7)
- added R146: 10kΩ, 1%, 63mW, reekilib_res:RESC1005, F.Cu at (93.2, 99.2)
- added R147: 0Ω, 5%, thin film, reekilib_res:RESC2012, F.Cu at (92.5, 95.0)
- added R148: 316kΩ, 1%, 63mW, reekilib_res:RESC1005, F.Cu at (100.6, 102.0)
- added R149: 53.6kΩ, 1%, 63mW, reekilib_res:RESC1005, F.Cu at (98.9, 102.0)
- added R150: 37.4kΩ, 1%, 63mW, reekilib_res:RESC1005, F.Cu at (94.0, 106.5)
- added R151: 21kΩ, 1%, 63mW, reekilib_res:RESC1005, F.Cu at (100.6, 103.0)
- added R152: 105kΩ, 1%, 63mW, reekilib_res:RESC1005, F.Cu at (95.2, 102.0)
- added R153: 316kΩ, 1%, 63mW, reekilib_res:RESC1005, F.Cu at (94.0, 103.5)
- added R154: 53.6kΩ, 1%, 63mW, reekilib_res:RESC1005, F.Cu at (94.0, 104.5)
- added R155: 10kΩ, 1%, 63mW, reekilib_res:RESC1005, F.Cu at (95.0, 93.5)
- added R156: 1kΩ, 1%, 63mW, reekilib_res:RESC1005, F.Cu at (98.2, 90.5)
- added R157: 33Ω, 1%, 63mW, reekilib_res:RESC1005, F.Cu at (243.2, 93.2)
- added R158: 33Ω, 1%, 63mW, reekilib_res:RESC1005, F.Cu at (266.3, 118.0)
- added U21: LM5158, reekilib_qfn:QFN50P300X300-17, F.Cu at (97.8, 104.8)
- added U22: TPS7A4001, reekilib_sop:SOP65P490X300-9, F.Cu at (97.0, 98.5)
- C108, C89, C92, R63: moved to B.Cu
- C115, C116: value 100nF, 16V, X7R -> 100nF, 25V, X7R
- D10, D11, D12, D13, D14, D15, D16, D6, D7, D8, D9: footprint reekilib_dfn:DFN50P100X250X55-10 -> reekilib_dfn:DFN50P100X250X55-10_ESD204
- U13, U14: value - -> LDL212DR
- moved C105 67.6 mm to (30.0, 118.0)
- moved C107 54.9 mm to (82.0, 118.0)
- moved C108 48.6 mm to (82.0, 118.0), turned to -90 degrees
- moved J20 29.8 mm to (237.6, 85.8), turned to 180 degrees
- moved C94 27.5 mm to (45.5, 103.5), turned to -90 degrees
- moved C137 23.9 mm to (40.1, 76.5)
- moved R63 18.6 mm to (57.5, 106.3)
- moved C132 18.0 mm to (45.2, 81.1)
- moved R65 18.0 mm to (58.8, 112.8), turned to -90 degrees
- moved R91 17.8 mm to (45.5, 79.5), turned to 180 degrees
- moved R92 17.8 mm to (42.2, 77.8)
- moved R90 17.8 mm to (42.2, 79.5), turned to 0 degrees
- moved C128 17.8 mm to (42.2, 87.8)
- moved C129 17.8 mm to (45.2, 87.8)
- moved C130 17.8 mm to (40.0, 84.5)
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Connections:
- net Net-(J1-TMDS.CLK+) renamed /Display/_HDMI.CLK+
- net Net-(J1-TMDS.CLK-) renamed /Display/_HDMI.CLK-
- net Net-(J1-TMDS.D0+) renamed /Display/_HDMI.D0+
- net Net-(J1-TMDS.D0-) renamed /Display/_HDMI.D0-
- net Net-(J1-TMDS.D1+) renamed /Display/_HDMI.D1+
- net Net-(J1-TMDS.D1-) renamed /Display/_HDMI.D1-
- net Net-(J1-TMDS.D2+) renamed /Display/_HDMI.D2+
- net Net-(J1-TMDS.D2-) renamed /Display/_HDMI.D2-
- C10 pad 2: Net-(C10-Pad2) -> /Real-Time MCU/MCU/VIO
- C11 pad 2: Net-(C11-Pad2) -> /Mgmt MCU/MCU/VIO
- C116 pad 1: VSSISO -> VSS
- C12 pad 2: Net-(C10-Pad2) -> /Real-Time MCU/MCU/VIO
- C13 pad 2: Net-(C11-Pad2) -> /Mgmt MCU/MCU/VIO
- C14 pad 2: Net-(C10-Pad2) -> /Real-Time MCU/MCU/VIO
- C15 pad 2: Net-(C11-Pad2) -> /Mgmt MCU/MCU/VIO
- C16 pad 2: Net-(C10-Pad2) -> /Real-Time MCU/MCU/VIO
- C17 pad 2: Net-(C11-Pad2) -> /Mgmt MCU/MCU/VIO
- C18 pad 2: Net-(C10-Pad2) -> /Real-Time MCU/MCU/VIO
- C19 pad 2: Net-(C11-Pad2) -> /Mgmt MCU/MCU/VIO
- C20 pad 2: Net-(C10-Pad2) -> /Real-Time MCU/MCU/VIO
- C21 pad 2: Net-(C11-Pad2) -> /Mgmt MCU/MCU/VIO
- C22 pad 2: Net-(C10-Pad2) -> /Real-Time MCU/MCU/VIO
- C23 pad 2: Net-(C11-Pad2) -> /Mgmt MCU/MCU/VIO
- C24 pad 2: Net-(C10-Pad2) -> /Real-Time MCU/MCU/VIO
- C25 pad 2: Net-(U3A-ADC.AVDD) -> /Mgmt MCU/MCU/VIO
- C26 pad 2: Net-(U4A-ADC.AVDD) -> /Real-Time MCU/MCU/VIO
- C27 pad 2: Net-(C27-Pad2) -> /Mgmt MCU/MCU/VCORE
- C28 pad 2: Net-(C28-Pad2) -> /Real-Time MCU/MCU/VCORE
- C29 pad 2: Net-(C27-Pad2) -> /Mgmt MCU/MCU/VCORE
- C3 pad 2: Net-(U5-VCC) -> /Mgmt MCU/MCU/VIO
- C30 pad 2: Net-(C28-Pad2) -> /Real-Time MCU/MCU/VCORE
- C31 pad 2: Net-(C27-Pad2) -> /Mgmt MCU/MCU/VCORE
- C32 pad 2: Net-(C28-Pad2) -> /Real-Time MCU/MCU/VCORE
- C4 pad 2: Net-(U6-VCC) -> /Real-Time MCU/MCU/VIO
- C5 pad 2: Net-(U3B-USB_OTP.VDD) -> /Mgmt MCU/MCU/VIO
- C6 pad 2: Net-(U4B-USB_OTP.VDD) -> /Real-Time MCU/MCU/VIO
- C7 pad 2: Net-(U3B-QSPI.IOVDD) -> /Mgmt MCU/MCU/VIO
- C8 pad 2: Net-(U4B-QSPI.IOVDD) -> /Real-Time MCU/MCU/VIO
- C9 pad 2: Net-(C11-Pad2) -> /Mgmt MCU/MCU/VIO
- R122 pad 2: VPHANTOM -> Net-(JMP3-Pad2)
- R123 pad 2: VPHANTOM -> Net-(JMP3-Pad2)
- R124 pad 2: VPHANTOM -> Net-(J26-Pad2)
- R125 pad 2: VPHANTOM -> Net-(J26-Pad2)
- R45 pad 1: /Real-Time MCU/RTIO.DIO0 -> /Real-Time MCU/RTIO.DIO7
- R45 pad 2: /Real-Time MCU/RTIO.DIO1 -> /Real-Time MCU/RTIO.DIO6
- R45 pad 3: /Real-Time MCU/RTIO.DIO2 -> /Real-Time MCU/RTIO.DIO5
- R45 pad 4: /Real-Time MCU/RTIO.DIO3 -> /Real-Time MCU/RTIO.DIO4
- R47 pad 1: /Real-Time MCU/RTIO.DIO4 -> /Real-Time MCU/RTIO.DIO3
- R47 pad 2: /Real-Time MCU/RTIO.DIO5 -> /Real-Time MCU/RTIO.DIO2
- R47 pad 3: /Real-Time MCU/RTIO.DIO6 -> /Real-Time MCU/RTIO.DIO1
- R47 pad 4: /Real-Time MCU/RTIO.DIO7 -> /Real-Time MCU/RTIO.DIO0
- U3 pad 10: Net-(C27-Pad2) -> /Mgmt MCU/MCU/VCORE
- U3 pad 15: Net-(C11-Pad2) -> /Mgmt MCU/MCU/VIO
- U3 pad 24: Net-(C11-Pad2) -> /Mgmt MCU/MCU/VIO
- U3 pad 29: Net-(C11-Pad2) -> /Mgmt MCU/MCU/VIO
- U3 pad 32: Net-(C27-Pad2) -> /Mgmt MCU/MCU/VCORE
- U3 pad 41: Net-(C11-Pad2) -> /Mgmt MCU/MCU/VIO
- U3 pad 5: Net-(C11-Pad2) -> /Mgmt MCU/MCU/VIO
- U3 pad 50: Net-(C11-Pad2) -> /Mgmt MCU/MCU/VIO
- U3 pad 51: Net-(C27-Pad2) -> /Mgmt MCU/MCU/VCORE
- U3 pad 59: Net-(U3A-ADC.AVDD) -> /Mgmt MCU/MCU/VIO
- U3 pad 60: Net-(C11-Pad2) -> /Mgmt MCU/MCU/VIO
- U3 pad 61: unconnected-(U3A-VREG.AVDD-Pad61) -> Net-(U3A-VREG.AVDD)
- U3 pad 63: unconnected-(U3A-VREG.LX-Pad63) -> Net-(U3A-VREG.LX)
- U3 pad 64: unconnected-(U3A-VREG.VIN-Pad64) -> /Mgmt MCU/MCU/VIO
- U3 pad 65: unconnected-(U3A-VREG.FB-Pad65) -> /Mgmt MCU/MCU/VCORE
- U3 pad 68: Net-(U3B-USB_OTP.VDD) -> /Mgmt MCU/MCU/VIO
- U3 pad 69: Net-(U3B-QSPI.IOVDD) -> /Mgmt MCU/MCU/VIO
- U3 pad 76: Net-(C11-Pad2) -> /Mgmt MCU/MCU/VIO
- U4 pad 10: Net-(C28-Pad2) -> /Real-Time MCU/MCU/VCORE
- U4 pad 15: Net-(C10-Pad2) -> /Real-Time MCU/MCU/VIO
- U4 pad 24: Net-(C10-Pad2) -> /Real-Time MCU/MCU/VIO
- U4 pad 29: Net-(C10-Pad2) -> /Real-Time MCU/MCU/VIO
- U4 pad 32: Net-(C28-Pad2) -> /Real-Time MCU/MCU/VCORE
- U4 pad 41: Net-(C10-Pad2) -> /Real-Time MCU/MCU/VIO
- U4 pad 5: Net-(C10-Pad2) -> /Real-Time MCU/MCU/VIO
- U4 pad 50: Net-(C10-Pad2) -> /Real-Time MCU/MCU/VIO
- U4 pad 51: Net-(C28-Pad2) -> /Real-Time MCU/MCU/VCORE
- U4 pad 59: Net-(U4A-ADC.AVDD) -> /Real-Time MCU/MCU/VIO
- U4 pad 60: Net-(C10-Pad2) -> /Real-Time MCU/MCU/VIO
- U4 pad 61: unconnected-(U4A-VREG.AVDD-Pad61) -> Net-(U4A-VREG.AVDD)
- U4 pad 63: unconnected-(U4A-VREG.LX-Pad63) -> Net-(U4A-VREG.LX)
- U4 pad 64: unconnected-(U4A-VREG.VIN-Pad64) -> /Real-Time MCU/MCU/VIO
- U4 pad 65: unconnected-(U4A-VREG.FB-Pad65) -> /Real-Time MCU/MCU/VCORE
- U4 pad 68: Net-(U4B-USB_OTP.VDD) -> /Real-Time MCU/MCU/VIO
- U4 pad 69: Net-(U4B-QSPI.IOVDD) -> /Real-Time MCU/MCU/VIO
- U4 pad 76: Net-(C10-Pad2) -> /Real-Time MCU/MCU/VIO
- U5 pad 8: Net-(U5-VCC) -> /Mgmt MCU/MCU/VIO
- U6 pad 8: Net-(U6-VCC) -> /Real-Time MCU/MCU/VIO
Routing:
- net VSS: track 2.15 -> 213.1 mm, vias 0 -> 83
- net VSSISO: track 0.00 -> 145.7 mm, vias 0 -> 58
- net V12ISO: track 0.00 -> 86.0 mm
- net /Real-Time MCU/MCU/VIO: track 0.00 -> 69.4 mm, vias 0 -> 10
- net /Mgmt MCU/MCU/VIO: track 0.00 -> 69.4 mm, vias 0 -> 10
- net /Audio/Audio inputs/MICLINE1.SIG-: track 2.83 -> 67.1 mm, vias 0 -> 1
- net /Audio/Audio inputs/MICLINE1.SIG+: track 2.83 -> 66.5 mm, vias 0 -> 1
- net /Mgmt MCU/MCU/VCORE: track 0.00 -> 40.8 mm, vias 0 -> 4
- net /Real-Time MCU/MCU/VCORE: track 0.00 -> 40.8 mm, vias 0 -> 4
- net VRTIO: track 0.00 -> 40.6 mm
- net V50: track 0.00 -> 39.3 mm
- net /Real-Time MCU/RTIO.DIO7: track 0.00 -> 27.7 mm
- net /Real-Time MCU/RTIO.DIO6: track 0.00 -> 26.3 mm
- net /Audio/Audio inputs/MICLINE2.SIG+: track 4.81 -> 31.0 mm, vias 0 -> 1
- net /Audio/Audio inputs/MICLINE2.SIG-: track 4.81 -> 30.4 mm, vias 0 -> 1
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