File: hw/pandore/pandore-audio-codec.kicad_sch (KiCad schematic)
At the start: 15 parts, among them U11 CS4272, X5 ${F}, ${tol}+${stab}, ${load}

Commit message: lots of work done all around
Parts:
- added R106, R107, R108, R109: ${Resistance}, ${Tolerance}, ${Power}, reekilib_res:RESC1005, symbol reekilib_res:res
Connections:
- net AVIO: no longer C90.2, C91.2, C92.2, U11.10 (VL), U11.9 (VD)
- net AVSS: now also R107.2, R109.2
- net ~{MUTE}.L: now also R106.2, R107.1
- net ~{MUTE}.R: now also R108.2, R109.1
- net AV5: now reaches C88.2, C89.2, U11.20 (VA)
- net AV5: now also R106.1, R108.1
- net VCM: now reaches C95.2, U11.15 (VCOM)
- net VSS renamed VSSISO
- new net AV3P3: C90.2, C91.2, C92.2, U11.10 (VL), U11.9 (VD)

Commit message: added i2s/i2c isolation for audio section
Connections:
- net AVIO is gone; now on net AV3P3: R64.1
- net CTL.~{RST} renamed ~{RST}
Changed lines of the file:
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@@
 	)
 	(bus_entry
-		(at 59.69 63.5)
-		(size 2.54 2.54)
-		(stroke
-			(width 0)
-			(type default)
-		)
-	)
-	(bus_entry
 		(at 59.69 52.07)
 		(size 2.54 2.54)
@@
 	(wire
 		(pts
+			(xy 57.15 66.04) (xy 140.97 66.04)
+		)
+		(stroke
+			(width 0)
+			(type default)
+		)
+	)
+	(wire
+		(pts
 			(xy 140.97 118.11) (xy 139.7 118.11)
 		)
@@
 	(bus
 		(pts
-			(xy 57.15 63.5) (xy 59.69 63.5)
+			(xy 57.15 72.39) (xy 59.69 72.39)
 		)
 		(stroke
@@
 	(wire
 		(pts
-			(xy 62.23 66.04) (xy 140.97 66.04)
-		)
-		(stroke
-			(width 0)
-			(type default)
-		)
-	)
-	(wire
-		(pts
 			(xy 173.99 85.09) (xy 194.31 85.09)
 		)
@@
 		)
 	)
-	(bus
-		(pts
-			(xy 59.69 63.5) (xy 59.69 72.39)
-		)
-		(stroke
-			(width 0)
-			(type default)
-		)
-	)
 	(wire
 		(pts
@@
 		)
 	)
-	(label "CTL.~{RST}"
-		(at 64.77 66.04 0)
-		(effects
-			(font
-				(size 1.016 1.016)
-			)
-			(justify left bottom)
-		)
-	)
 	(label "MICLINE1.SIG-"
 		(at 179.07 80.01 0)
@@
 		)
 	)
-	(hierarchical_label "CTL{I2C ~{RST}}"
+	(hierarchical_label "CTL{I2C}"
 		(shape bidirectional)
-		(at 57.15 63.5 180)
+		(at 57.15 72.39 180)
 		(effects
 			(font
@@
 		)
 	)
+	(hierarchical_label "~{RST}"
+		(shape input)
+		(at 57.15 66.04 180)
+		(effects
+			(font
+				(size 1.016 1.016)
+			)
+			(justify right)
+		)
+	)
 	(hierarchical_label "VCM"
 		(shape output)
@@
 	)
 	(symbol
+		(lib_id "reekilib_pwr:VDD")
+		(at 85.09 91.44 0)
+		(unit 1)
+		(exclude_from_sim no)
+		(in_bom no)
+		(on_board no)
+		(dnp no)
+		(property "Reference" "#PWR0111"
+			(at 85.09 88.265 0)
+			(do_not_autoplace yes)
+			(effects
+				(font
+					(size 1 1)
+				)
+				(hide yes)
+			)
+		)
+		(property "Value" "AV3P3"
+			(at 85.09 90.17 0)
+			(effects
+				(font
+					(size 1 1)
+				)
+			)
+		)
+		(property "Footprint" ""
+			(at 85.09 91.44 0)
+			(effects
+				(font
+					(size 1.524 1.524)
+				)
+			)
+		)
+		(property "Datasheet" ""
+			(at 85.09 91.44 0)
+			(effects
+				(font
+					(size 1.524 1.524)
+				)
+			)
+		)
+		(property "Description" ""
+			(at 85.09 91.44 0)
+			(effects
+				(font
+					(size 1.27 1.27)
+				)
+				(hide yes)
+			)
+		)
+		(pin "1"
+		)
+		(instances
+			(project "pandore"
+				(path "/e55f2700-f75a-4062-8a27-fe258faa8966/b4e2772d-7748-46ec-bd38-bc8e72cebcb8/c7a6c4ca-6083-4b1c-b07a-a9d1f5204bfb"
+					(reference "#PWR0111")
+					(unit 1)
+				)
+			)
+		)
+	)
+	(symbol
 		(lib_id "reekilib_pwr:VSS")
 		(at 139.7 134.62 0)
@@
 					(unit 1)
 				)
-			)
-		)
-	)
-	(symbol
-		(lib_id "reekilib_pwr:VDD")
-		(at 85.09 91.44 0)
-		(unit 1)
-		(exclude_from_sim no)
-		(in_bom no)
-		(on_board no)
-		(dnp no)
-		(property "Reference" "#PWR0111"
-			(at 85.09 88.265 0)
-			(do_not_autoplace yes)
-			(effects
-				(font
-					(size 1 1)
-				)
-				(hide yes)
-			)
-		)
-		(property "Value" "AVIO"
-			(at 85.09 90.17 0)
-			(effects
-				(font
-					(size 1 1)
-				)
-			)
-		)
-		(property "Footprint" ""
-			(at 85.09 91.44 0)
-			(effects
-				(font
-					(size 1.524 1.524)
-				)
-			)
-		)
-		(property "Datasheet" ""
-			(at 85.09 91.44 0)
-			(effects
-				(font
-					(size 1.524 1.524)
-				)
-			)
-		)
-		(property "Description" ""
-			(at 85.09 91.44 0)
-			(effects
-				(font
-					(size 1.27 1.27)
-				)
-				(hide yes)
-			)
-		)
-		(pin "1"
-		)
-		(instances
-			(project "pandore"
-				(path "/e55f2700-f75a-4062-8a27-fe258faa8966/b4e2772d-7748-46ec-bd38-bc8e72cebcb8/c7a6c4ca-6083-4b1c-b07a-a9d1f5204bfb"
-					(reference "#PWR0111")
-					(unit 1)
-				)

Commit message: most of board control signals added, routed and defined
Parts:
- added C235: ${Capacitance}, ${Voltage}, ${Dielectric}, reekilib_cap:CAPC1005, symbol reekilib_cap:cap
- added C236: ${Capacitance}, ${Voltage}, ${Dielectric}, reekilib_cap:CAPC2012, symbol reekilib_cap:cap
- added C237: ${Capacitance}, ${Voltage}, ${Dielectric}, reekilib_cap:CAPC1608, symbol reekilib_cap:cap
- added R204, R205: ${Resistance}, ${Tolerance}, ${Type}, reekilib_res:RESC2012, symbol reekilib_res:res
- added U26: OPAMP_2, reekilib_soic:SOIC127P600X150-8, symbol reekilib_amp:OPAMP_2
Connections:
- net AV5: now also C235.2, C236.2, U26.8 (V+)
- net AVSS: now also C235.1, C236.1, C237.1, U26.4 (V-)
- net VCM: no longer names the net of C95.2, U11.15 (VCOM)
- net VCM: now also C237.2, U26.3 (IN+), U26.5 (IN+)
- new net: R205.1, U26.6 (IN-), U26.7 (OUT)
- new net: R204.1, U26.1 (OUT), U26.2 (IN-)
- new net VCM1: R204.2
- new net VCM2: R205.2

Commit message: added monitor amp with volume knob continue routing all around
Parts:
- U26: value OPAMP_2 -> OPA1656; Link ? -> https://www.ti.com/product/OPA1656; MFG ? -> TI; MPN ? -> OPA1656IDR
Changed lines of the file:
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@@
 			)
 		)
-		(property "Value" "OPAMP_2"
+		(property "Value" "OPA1656"
 			(at 234.95 160.02 0)
 			(do_not_autoplace yes)
@@
 			)
 		)
-		(property "Datasheet" "?"
+		(property "Datasheet" "https://www.ti.com/lit/ds/symlink/opa1656.pdf"
 			(at 243.205 167.64 0)
 			(effects
@@
 			)
 		)
-		(property "MPN" "?"
+		(property "MPN" "OPA1656IDR"
 			(at 243.205 161.925 0)
 			(effects
@@
 			)
 		)
-		(property "MFG" "?"
+		(property "MFG" "TI"
 			(at 243.205 163.83 0)
 			(effects
@@
 			)
 		)
-		(property "Link" "?"
+		(property "Link" "https://www.ti.com/product/OPA1656"
 			(at 243.205 165.735 0)
 			(effects
@@
 			)
 		)
-		(property "Value" "OPAMP_2"
+		(property "Value" "OPA1656"
 			(at 234.95 130.81 0)
 			(do_not_autoplace yes)
@@
 			)
 		)
-		(property "Datasheet" "?"
+		(property "Datasheet" "https://www.ti.com/lit/ds/symlink/opa1656.pdf"
 			(at 243.205 138.43 0)
 			(effects
@@
 			)
 		)
-		(property "MPN" "?"
+		(property "MPN" "OPA1656IDR"
 			(at 243.205 132.715 0)
 			(effects
@@
 			)
 		)
-		(property "MFG" "?"
+		(property "MFG" "TI"
 			(at 243.205 134.62 0)
 			(effects
@@
 			)
 		)
-		(property "Link" "?"
+		(property "Link" "https://www.ti.com/product/OPA1656"
 			(at 243.205 136.525 0)
 			(effects

Commit message: last sprint almost done, most routing done
Parts:
- removed R63: ${Resistance}, ${Tolerance}, ${Power}, reekilib_res:RESC1005, symbol reekilib_res:res
Connections:
- net VSSISO is gone; now on net AVSS: C90.1, C91.1, C92.1, C96.1, C97.1, R65.2, U11.8 (DGND), X5.2, X5.4
- net VCM0: now reaches C237.2, C95.2, U11.15 (VCOM), U26.3 (IN+), U26.5 (IN+)
Changed lines of the file:
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@@
 	)
 	(junction
+		(at 207.01 100.33)
+		(diameter 0)
+		(color 0 0 0 0)
+	)
+	(junction
 		(at 191.77 116.84)
 		(diameter 0)
@@
 	(wire
 		(pts
-			(xy 161.29 132.08) (xy 175.26 132.08)
-		)
-		(stroke
-			(width 0)
-			(type default)
-		)
-	)
-	(wire
-		(pts
 			(xy 185.42 116.84) (xy 191.77 116.84)
 		)
@@
 	(wire
 		(pts
+			(xy 207.01 100.33) (xy 266.7 100.33)
+		)
+		(stroke
+			(width 0)
+			(type default)
+		)
+	)
+	(wire
+		(pts
 			(xy 245.11 143.51) (xy 245.11 154.94)
 		)
@@
 	(wire
 		(pts
-			(xy 139.7 132.08) (xy 153.67 132.08)
+			(xy 139.7 132.08) (xy 175.26 132.08)
 		)
 		(stroke
@@
 		)
 	)
+	(hierarchical_label "VCM0"
+		(shape output)
+		(at 266.7 100.33 0)
+		(effects
+			(font
+				(size 1.016 1.016)
+			)
+			(justify left)
+		)
+	)
 	(hierarchical_label "CTL{I2C}"
 		(shape bidirectional)
@@
 					(unit 1)
 				)
-			)
-		)
-	)
-	(symbol
-		(lib_id "reekilib_res:res")
-		(at 157.48 132.08 270)
-		(unit 1)
-		(exclude_from_sim no)
-		(in_bom yes)
-		(on_board yes)
-		(dnp no)
-		(property "Reference" "R63"
-			(at 159.385 134.62 90)
-			(do_not_autoplace yes)
-			(effects
-				(font
-					(size 1 1)
-				)
-				(justify right)
-			)
-		)
-		(property "Value" "${Resistance}, ${Tolerance}, ${Power}"
-			(at 158.242 134.112 0)
-			(do_not_autoplace yes)
-			(effects
-				(font
-					(size 1 1)
-				)
-				(justify left)
-				(hide yes)
-			)
-		)
-		(property "Footprint" "reekilib_res:RESC1005"
-			(at 146.304 132.334 0)
-			(do_not_autoplace yes)
-			(effects
-				(font
-					(size 1 1)
-				)
-				(hide yes)
-			)
-		)
-		(property "Datasheet" ""
-			(at 143.256 132.08 0)
-			(do_not_autoplace yes)
-			(effects
-				(font
-					(size 1 1)
-				)
-				(hide yes)
-			)
-		)
-		(property "Description" "Resistor single 2 pad"
-			(at 144.78 132.08 0)
-			(do_not_autoplace yes)
-			(effects
-				(font
-					(size 1 1)
-				)
-				(hide yes)
-			)
-		)
-		(property "Resistance" "0Ω"
-			(at 159.385 136.271 90)
-			(do_not_autoplace yes)
-			(effects
-				(font
-					(size 1 1)
-				)
-				(justify right)
-			)
-		)
-		(property "Tolerance" "5%"
-			(at 159.385 137.795 90)
-			(do_not_autoplace yes)
-			(effects
-				(font
-					(size 1 1)
-				)
-				(justify right)
-			)
-		)
-		(property "Power" "63mW"
-			(at 159.385 139.319 90)
-			(do_not_autoplace yes)
-			(effects
-				(font
-					(size 1 1)
-				)
-				(justify right)
-			)
-		)
-		(property "MPN" ""
-			(at 139.7 132.08 0)
-			(do_not_autoplace yes)
-			(effects
-				(font
-					(size 1 1)
-				)
-				(hide yes)
-			)
-		)
-		(property "MFG" ""
-			(at 139.954 146.05 0)
-			(do_not_autoplace yes)
-			(effects
-				(font
-					(size 1 1)
-				)
-				(justify left)
-				(hide yes)
-			)
-		)
-		(property "Link" ""
-			(at 141.732 132.334 0)
-			(do_not_autoplace yes)
-			(effects
-				(font
-					(size 1 1)
-				)
-				(hide yes)
-			)
-		)
-		(property "MPN2" ""
-			(at 137.922 131.572 0)
-			(do_not_autoplace yes)
-			(effects
-				(font
-					(size 1 1)
-				)
-				(hide yes)
-			)
-		)
-		(property "MFG2" ""
-			(at 137.922 146.304 0)
-			(do_not_autoplace yes)
-			(effects
-				(font
-					(size 1 1)
-				)
-				(justify left)
-				(hide yes)
-			)
-		)
-		(property "MPN3" ""
-			(at 136.144 132.08 0)
-			(do_not_autoplace yes)
-			(effects
-				(font
-					(size 1 1)
-				)
-				(hide yes)
-			)
-		)
-		(property "MFG3" ""
-			(at 136.144 146.304 0)
-			(do_not_autoplace yes)
-			(effects
-				(font
-					(size 1 1)
-				)
-				(justify left)
-				(hide yes)
-			)
-		)
-		(pin "2"
-		)
-		(pin "1"
-		)
-		(instances
-			(project "pandore"
-				(path "/e55f2700-f75a-4062-8a27-fe258faa8966/b4e2772d-7748-46ec-bd38-bc8e72cebcb8/c7a6c4ca-6083-4b1c-b07a-a9d1f5204bfb"
-					(reference "R63")
-					(unit 1)
-				)

Commit message: finished adding mpn,mfg to all parts, finished routing placement
Parts:
- C235, C88, C90, C91, C93, C95: MFG2 Samsung Electro-Mechanics -> (none); MFG3 Taiyo Yuden -> (none); MPN2 CL05B104KA5NNNC -> (none); MPN3 EMK105B7104KV-F -> (none); Voltage 16V -> 25V
- C236, C89, C92: MFG (none) -> Murata; MPN (none) -> GRM21BR61E106KA73K; Voltage 16V -> 25V
- C237: MFG (none) -> KEMET; MPN (none) -> C0603C105K4RACTU
- C96, C97: Link (none) -> https://yageogroup.com/products/Capacitors/part/CC0402JRNPO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; MFG (none) -> Yageo; MPN (none) -> CC0402JRNPO9BN120
- R204, R205: MFG (none) -> Stackpole Electronics Inc; MPN (none) -> RNCF0805DTE10R0; Power 0.25W -> 250mW
- R65: Link (none) -> https://yageogroup.com/products/Resistors/part/RC0402FR-131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; MFG (none) -> YAGEO; MPN (none) -> RC0402FR-131KL
Changed lines of the file:
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@@
 			)
 		)
-		(property "Datasheet" ""
+		(property "Datasheet" "https://mm.digikey.com/Volume0/opasdata/d220001/medias/docus/6536/ABM8_Datasheet.pdf"
 			(at 115.57 111.76 0)
 			(do_not_autoplace yes)
@@
 			)
 		)
-		(property "Voltage" "16V"
+		(property "Voltage" "25V"
 			(at 134.62 115.316 0)
 			(do_not_autoplace yes)
@@
 			)
 		)
-		(property "MPN2" "CL05B104KA5NNNC"
+		(property "MPN2" ""
 			(at 134.62 143.51 0)
 			(do_not_autoplace yes)
@@
 			)
 		)
-		(property "MFG2" "Samsung Electro-Mechanics"
+		(property "MFG2" ""
 			(at 146.558 143.51 0)
 			(do_not_autoplace yes)
@@
 			)
 		)
-		(property "MPN3" "EMK105B7104KV-F"
+		(property "MPN3" ""
 			(at 134.62 145.034 0)
 			(do_not_autoplace yes)
@@
 			)
 		)
-		(property "MFG3" "Taiyo Yuden"
+		(property "MFG3" ""
 			(at 146.558 145.034 0)
 			(do_not_autoplace yes)
@@
 			)
 		)
-		(property "Voltage" "16V"
+		(property "Voltage" "25V"
 			(at 231.14 110.109 0)
 			(do_not_autoplace yes)
@@
 			)
 		)
-		(property "MPN2" "CL05B104KA5NNNC"
+		(property "MPN2" ""
 			(at 231.14 135.89 0)
 			(do_not_autoplace yes)
@@
 			)
 		)
-		(property "MFG2" "Samsung Electro-Mechanics"
+		(property "MFG2" ""
 			(at 243.078 135.89 0)
 			(do_not_autoplace yes)
@@
 			)
 		)
-		(property "MPN3" "EMK105B7104KV-F"
+		(property "MPN3" ""
 			(at 231.14 137.414 0)
 			(do_not_autoplace yes)
@@
 			)
 		)
-		(property "MFG3" "Taiyo Yuden"
+		(property "MFG3" ""
 			(at 243.078 137.414 0)
 			(do_not_autoplace yes)
@@
 			)
 		)
-		(property "Voltage" "16V"
+		(property "Voltage" "25V"
 			(at 175.26 117.729 0)
 			(do_not_autoplace yes)
@@
 			)
 		)
-		(property "MPN2" "CL05B104KA5NNNC"
+		(property "MPN2" ""
 			(at 175.26 143.51 0)
 			(do_not_autoplace yes)
@@
 			)
 		)
-		(property "MFG2" "Samsung Electro-Mechanics"
+		(property "MFG2" ""
 			(at 187.198 143.51 0)
 			(do_not_autoplace yes)
@@
 			)
 		)
-		(property "MPN3" "EMK105B7104KV-F"
+		(property "MPN3" ""
 			(at 175.26 145.034 0)
 			(do_not_autoplace yes)
@@
 			)
 		)
-		(property "MFG3" "Taiyo Yuden"
+		(property "MFG3" ""
 			(at 187.198 145.034 0)
 			(do_not_autoplace yes)
@@
 			)
 		)
-		(property "Voltage" "16V"
+		(property "Voltage" "25V"
 			(at 185.42 107.569 0)
 			(do_not_autoplace yes)
@@
 			)
 		)
-		(property "MPN2" "CL05B104KA5NNNC"
+		(property "MPN2" ""
 			(at 185.42 133.35 0)
 			(do_not_autoplace yes)
@@
 			)
 		)
-		(property "MFG2" "Samsung Electro-Mechanics"
+		(property "MFG2" ""
 			(at 197.358 133.35 0)
 			(do_not_autoplace yes)
@@
 			)
 		)
-		(property "MPN3" "EMK105B7104KV-F"
+		(property "MPN3" ""
 			(at 185.42 134.874 0)
 			(do_not_autoplace yes)
@@
 			)
 		)
-		(property "MFG3" "Taiyo Yuden"
+		(property "MFG3" ""
 			(at 197.358 134.874 0)
 			(do_not_autoplace yes)
@@
 			)
 		)
-		(property "Datasheet" ""
+		(property "Datasheet" "https://search.murata.co.jp/Ceramy/image/img/A01X/G101/ENG/GRM21BR61E106KA73-01.pdf"
 			(at 236.22 130.048 0)
 			(do_not_autoplace yes)
@@
 			)
 		)
-		(property "Voltage" "16V"
+		(property "Voltage" "25V"
 			(at 236.22 110.109 0)
 			(do_not_autoplace yes)
@@
 			)
 		)
-		(property "MPN" ""
+		(property "MPN" "GRM21BR61E106KA73K"
 			(at 236.22 134.366 0)
 			(do_not_autoplace yes)
@@
 			)
 		)
-		(property "MFG" ""
+		(property "MFG" "Murata"
 			(at 248.158 134.366 0)
 			(do_not_autoplace yes)
@@
 			)
 		)
-		(property "Voltage" "16V"
+		(property "Voltage" "25V"
 			(at 139.7 115.316 0)
 			(do_not_autoplace yes)
@@
 			)
 		)
-		(property "MPN2" "CL05B104KA5NNNC"
+		(property "MPN2" ""
 			(at 139.7 143.51 0)
 			(do_not_autoplace yes)
@@
 			)
 		)
-		(property "MFG2" "Samsung Electro-Mechanics"
+		(property "MFG2" ""
 			(at 151.638 143.51 0)
 			(do_not_autoplace yes)
@@
 			)
 		)
-		(property "MPN3" "EMK105B7104KV-F"
+		(property "MPN3" ""
 			(at 139.7 145.034 0)
 			(do_not_autoplace yes)
@@
 			)
 		)
-		(property "MFG3" "Taiyo Yuden"
+		(property "MFG3" ""
 			(at 151.638 145.034 0)
 			(do_not_autoplace yes)
@@
 			)
 		)
-		(property "Datasheet" ""
+		(property "Datasheet" "https://search.murata.co.jp/Ceramy/image/img/A01X/G101/ENG/GRM21BR61E106KA73-01.pdf"
 			(at 129.54 137.668 0)
 			(do_not_autoplace yes)
@@
 			)
 		)
-		(property "Voltage" "16V"
+		(property "Voltage" "25V"
 			(at 129.54 117.729 0)
 			(do_not_autoplace yes)
@@
 			)
 		)
-		(property "MPN" ""
+		(property "MPN" "GRM21BR61E106KA73K"
 			(at 129.54 141.986 0)
 			(do_not_autoplace yes)
@@
 			)
 		)
-		(property "MFG" ""
+		(property "MFG" "Murata"
 			(at 141.478 141.986 0)
 			(do_not_autoplace yes)
@@
 			)
 		)
-		(property "Datasheet" ""
+		(property "Datasheet" "https://search.murata.co.jp/Ceramy/image/img/A01X/G101/ENG/GRM21BR61E106KA73-01.pdf"
 			(at 180.34 137.668 0)
 			(do_not_autoplace yes)
@@
 			)
 		)
-		(property "Voltage" "16V"
+		(property "Voltage" "25V"
 			(at 180.34 117.729 0)
 			(do_not_autoplace yes)
@@
 			)
 		)
-		(property "MPN" ""
+		(property "MPN" "GRM21BR61E106KA73K"
 			(at 180.34 141.986 0)
 			(do_not_autoplace yes)
@@
 			)
 		)
-		(property "MFG" ""
+		(property "MFG" "Murata"
 			(at 192.278 141.986 0)
 			(do_not_autoplace yes)
@@
 			)
 		)
-		(property "Datasheet" ""
+		(property "Datasheet" "https://yageogroup.com/content/datasheet/asset/file/UPY-GP_NP0_16V-to-250V"
 			(at 121.92 113.538 0)
 			(do_not_autoplace yes)
@@
 			)
 		)
-		(property "MPN" ""
+		(property "MPN" "CC0402JRNPO9BN120"
 			(at 121.92 117.856 0)
 			(do_not_autoplace yes)
@@
 			)
 		)
-		(property "MFG" ""
+		(property "MFG" "Yageo"
 			(at 133.858 117.856 0)
 			(do_not_autoplace yes)
@@
 			)
 		)
-		(property "Link" ""
+		(property "Link" "https://yageogroup.com/products/Capacitors/part/CC0402JRNPO9BN120"
 			(at 121.92 112.014 0)
 			(do_not_autoplace yes)
@@
 			)
 		)
-		(property "Datasheet" ""
+		(property "Datasheet" "https://yageogroup.com/content/datasheet/asset/file/PYU-RC_GROUP_51_ROHS_L"
 			(at 85.09 120.904 0)
 			(do_not_autoplace yes)
@@
 			)
 		)
-		(property "Link" ""
+		(property "Link" "https://yageogroup.com/products/Resistors/part/RC0402FR-131KL"
 			(at 85.344 122.428 0)
 			(do_not_autoplace yes)
@@
 			)
 		)
-		(property "MPN" ""
+		(property "MPN" "RC0402FR-131KL"
 			(at 85.09 124.46 0)
 			(do_not_autoplace yes)
@@
 			)
 		)
-		(property "MFG" ""
+		(property "MFG" "YAGEO"
 			(at 99.06 124.206 0)
 			(do_not_autoplace yes)
@@
 			)
 		)
-		(property "Datasheet" ""
+		(property "Datasheet" "https://yageogroup.com/content/datasheet/asset/file/KEM_C1002_X7R_SMD"
 			(at 180.34 117.348 0)
 			(do_not_autoplace yes)
@@
 			)
 		)
-		(property "MPN" ""
+		(property "MPN" "C0603C105K4RACTU"
 			(at 180.34 121.666 0)
 			(do_not_autoplace yes)
@@
 			)
 		)
-		(property "MFG" ""
+		(property "MFG" "KEMET"
 			(at 192.278 121.666 0)
 			(do_not_autoplace yes)
@@
 			)
 		)
-		(property "Voltage" "16V"
+		(property "Voltage" "25V"
 			(at 175.26 97.409 0)
 			(do_not_autoplace yes)
@@
 			)
 		)
-		(property "MPN2" "CL05B104KA5NNNC"
+		(property "MPN2" ""
 			(at 175.26 123.19 0)
 			(do_not_autoplace yes)
@@
 			)
 		)
-		(property "MFG2" "Samsung Electro-Mechanics"
+		(property "MFG2" ""
 			(at 187.198 123.19 0)
 			(do_not_autoplace yes)
@@
 			)
 		)
-		(property "MPN3" "EMK105B7104KV-F"
+		(property "MPN3" ""
 			(at 175.26 124.714 0)
 			(do_not_autoplace yes)
@@
 			)
 		)
-		(property "MFG3" "Taiyo Yuden"
+		(property "MFG3" ""
 			(at 187.198 124.714 0)
 			(do_not_autoplace yes)
@@
 			)
 		)
-		(property "Datasheet" ""
+		(property "Datasheet" "https://www.seielect.com/catalog/SEI-RNCF.pdf"
 			(at 268.224 154.94 0)
 			(do_not_autoplace yes)
@@
 			)
 		)
-		(property "Power" "0.25W"
+		(property "Power" "250mW"
 			(at 254 153.035 90)
 			(do_not_autoplace yes)
@@
 			)
 		)
-		(property "MPN" ""
+		(property "MPN" "RNCF0805DTE10R0"
 			(at 271.78 154.94 0)
 			(do_not_autoplace yes)
@@
 			)
 		)
-		(property "MFG" ""
+		(property "MFG" "Stackpole Electronics Inc"
 			(at 271.526 140.97 0)
 			(do_not_autoplace yes)
@@
 			)
 		)
-		(property "Datasheet" ""
+		(property "Datasheet" "https://www.seielect.com/catalog/SEI-RNCF.pdf"
 			(at 268.224 125.73 0)
 			(do_not_autoplace yes)
@@
 			)
 		)
-		(property "Power" "0.25W"
+		(property "Power" "250mW"
 			(at 254 123.825 90)
 			(do_not_autoplace yes)
@@
 			)
 		)
-		(property "MPN" ""
+		(property "MPN" "RNCF0805DTE10R0"
 			(at 271.78 125.73 0)
 			(do_not_autoplace yes)
@@
 			)
 		)
-		(property "MFG" ""
+		(property "MFG" "Stackpole Electronics Inc"
 			(at 271.526 111.76 0)
 			(do_not_autoplace yes)
@@
 			)
 		)
-		(property "Datasheet" ""
+		(property "Datasheet" "https://yageogroup.com/content/datasheet/asset/file/UPY-GP_NP0_16V-to-250V"
 			(at 109.22 113.538 0)
 			(do_not_autoplace yes)
@@
 			)
 		)
-		(property "MPN" ""
+		(property "MPN" "CC0402JRNPO9BN120"
 			(at 109.22 117.856 0)
 			(do_not_autoplace yes)
@@
 			)
 		)
-		(property "MFG" ""
+		(property "MFG" "Yageo"
 			(at 97.282 117.856 0)
 			(do_not_autoplace yes)
@@
 			)
 		)
-		(property "Link" ""
+		(property "Link" "https://yageogroup.com/products/Capacitors/part/CC0402JRNPO9BN120"
 			(at 109.22 112.014 0)
 			(do_not_autoplace yes)
