File: hw/pandore/pandore-audio-monitor.kicad_sch (KiCad schematic)
At the start: 37 parts, among them U34 OPA1656, U35 OPA1656, U36 OPA1656

Commit message: finished adding mpn,mfg to all parts, finished routing placement
Parts:
- C279, C283, C285: MFG2 Samsung Electro-Mechanics -> (none); MFG3 Taiyo Yuden -> (none); MPN2 CL05B104KA5NNNC -> (none); MPN3 EMK105B7104KV-F -> (none); Voltage 16V -> 25V
- C280, C284, C286: MFG (none) -> Murata; MPN (none) -> GRM21BR61E106KA73K; Voltage 16V -> 25V
- C281, C282, C287, C288: MFG (none) -> Walsin Technology Corporation; MPN (none) -> 0603N301J500CT
- R252, R253, R258, R259, R262, R263, R264, R266, R267, R269: Link (none) -> https://yageogroup.com/products/Resistors/part/RT0805DRE075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
- R254, R255, R256, R257: MFG (none) -> Susumu; MPN (none) -> RR1220P-103-D
- R260, R261, R270, R274, R275: Link (none) -> https://yageogroup.com/products/Resistors/part/RT0805DRE074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; MFG (none) -> YAGEO; MPN (none) -> RC0805JR-070RL; Power 0.25W -> 250mW
- R265, R268, R271, R272: MFG (none) -> Stackpole Electronics Inc; MPN (none) -> RNCF0805DTE10R0; Power 0.25W -> 250mW
- R273: Resistance (none) -> 10kΩ
