File: hw/pandore/pandore-bootctl.kicad_sch (KiCad schematic)
At the start: 29 parts, among them J30 PWRBTN, J31 RSTBTN, Q11 MOSFET_EN-N, Q12 MOSFET_EN-N, Q13 MOSFET_EN-N, Q14 MOSFET_EN-N, Q15 MOSFET_EN-N

Commit message: finished adding mpn,mfg to all parts, finished routing placement
Parts:
- C238, C239: MFG (none) -> KEMET; MPN (none) -> C0603C105K4RACTU
- C258: MFG (none) -> Murata; MPN (none) -> GRM21BR61E106KA73K
- J30, J31, JMP12: MFG (none) -> Adam Tech; MPN (none) -> PH1-02-UA
- JMP15: Link url-link -> (none); MFG MFG -> Adam Tech; MPN MPN -> PH1-03-UA
- R209, R210: Link (none) -> https://yageogroup.com/products/Resistors/part/RC0402FR-074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; MFG (none) -> YAGEO; MPN (none) -> RC0402FR-0749R9L
- R218, R220, R229, R230: Link (none) -> https://yageogroup.com/products/Resistors/part/RC0402FR-131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; MFG (none) -> YAGEO; MPN (none) -> RC0402FR-131KL
- R221: Link (none) -> https://yageogroup.com/products/Resistors/part/RC0402FR-079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; MFG (none) -> YAGEO; MPN (none) -> RC0402FR-07100KL
- R222: Link (none) -> https://yageogroup.com/products/Resistors/part/RC0402FR-071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; MFG (none) -> YAGEO; MPN (none) -> RC0402FR-071ML
Changed lines of the file:
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@@
 			)
 		)
-		(property "Datasheet" ""
+		(property "Datasheet" "https://yageogroup.com/content/datasheet/asset/file/KEM_C1002_X7R_SMD"
 			(at 86.36 164.338 0)
 			(do_not_autoplace yes)
@@
 			)
 		)
-		(property "MPN" ""
+		(property "MPN" "C0603C105K4RACTU"
 			(at 86.36 168.656 0)
 			(do_not_autoplace yes)
@@
 			)
 		)
-		(property "MFG" ""
+		(property "MFG" "KEMET"
 			(at 98.298 168.656 0)
 			(do_not_autoplace yes)
@@
 			)
 		)
-		(property "Datasheet" ""
+		(property "Datasheet" "https://search.murata.co.jp/Ceramy/image/img/A01X/G101/ENG/GRM21BR61E106KA73-01.pdf"
 			(at 58.42 124.968 0)
 			(do_not_autoplace yes)
@@
 			)
 		)
-		(property "MPN" ""
+		(property "MPN" "GRM21BR61E106KA73K"
 			(at 58.42 129.286 0)
 			(do_not_autoplace yes)
@@
 			)
 		)
-		(property "MFG" ""
+		(property "MFG" "Murata"
 			(at 70.358 129.286 0)
 			(do_not_autoplace yes)
@@
 			)
 		)
-		(property "Datasheet" ""
+		(property "Datasheet" "https://yageogroup.com/content/datasheet/asset/file/KEM_C1002_X7R_SMD"
 			(at 86.36 140.208 0)
 			(do_not_autoplace yes)
@@
 			)
 		)
-		(property "MPN" ""
+		(property "MPN" "C0603C105K4RACTU"
 			(at 86.36 144.526 0)
 			(do_not_autoplace yes)
@@
 			)
 		)
-		(property "MFG" ""
+		(property "MFG" "KEMET"
 			(at 98.298 144.526 0)
 			(do_not_autoplace yes)
@@
 			)
 		)
-		(property "Datasheet" ""
+		(property "Datasheet" "https://yageogroup.com/content/datasheet/asset/file/PYU-RC_GROUP_51_ROHS_L"
 			(at 112.014 121.92 0)
 			(do_not_autoplace yes)
@@
 			)
 		)
-		(property "MPN" ""
+		(property "MPN" "RC0402FR-0749R9L"
 			(at 115.57 121.92 0)
 			(do_not_autoplace yes)
@@
 			)
 		)
-		(property "MFG" ""
+		(property "MFG" "YAGEO"
 			(at 115.316 107.95 0)
 			(do_not_autoplace yes)
@@
 			)
 		)
-		(property "Link" ""
+		(property "Link" "https://yageogroup.com/products/Resistors/part/RC0402FR-0749R9L"
 			(at 115.57 78.105 0)
 			(do_not_autoplace yes)
@@
 			)
 		)
-		(property "Datasheet" ""
+		(property "Datasheet" "https://app.adam-tech.com/products/download/data_sheet/201605/ph1-xx-ua-data-sheet.pdf"
 			(at 58.42 113.284 0)
 			(do_not_autoplace yes)
@@
 			)
 		)
-		(property "MPN" ""
+		(property "MPN" "PH1-02-UA"
 			(at 58.42 119.126 0)
 			(do_not_autoplace yes)
@@
 			)
 		)
-		(property "MFG" ""
+		(property "MFG" "Adam Tech"
 			(at 51.816 119.126 0)
 			(do_not_autoplace yes)
@@
 			)
 		)
-		(property "Datasheet" ""
+		(property "Datasheet" "https://yageogroup.com/content/datasheet/asset/file/PYU-RC_GROUP_51_ROHS_L"
 			(at 73.66 110.744 0)
 			(do_not_autoplace yes)
@@
 			)
 		)
-		(property "Link" ""
+		(property "Link" "https://yageogroup.com/products/Resistors/part/RC0402FR-0793K1L"
 			(at 73.914 112.268 0)
 			(do_not_autoplace yes)
@@
 			)
 		)
-		(property "MPN" ""
+		(property "MPN" "RC0402FR-07100KL"
 			(at 73.66 114.3 0)
 			(do_not_autoplace yes)
@@
 			)
 		)
-		(property "MFG" ""
+		(property "MFG" "YAGEO"
 			(at 87.63 114.046 0)
 			(do_not_autoplace yes)
@@
 			)
 		)
-		(property "Datasheet" ""
+		(property "Datasheet" "https://yageogroup.com/content/datasheet/asset/file/PYU-RC_GROUP_51_ROHS_L"
 			(at 64.77 78.994 0)
 			(do_not_autoplace yes)
@@
 			)
 		)
-		(property "Link" ""
+		(property "Link" "https://yageogroup.com/products/Resistors/part/RC0402FR-131KL"
 			(at 65.024 80.518 0)
 			(do_not_autoplace yes)
@@
 			)
 		)
-		(property "MPN" ""
+		(property "MPN" "RC0402FR-131KL"
 			(at 64.77 82.55 0)
 			(do_not_autoplace yes)
@@
 			)
 		)
-		(property "MFG" ""
+		(property "MFG" "YAGEO"
 			(at 78.74 82.296 0)
 			(do_not_autoplace yes)
@@
 			)
 		)
-		(property "Datasheet" ""
+		(property "Datasheet" "https://yageogroup.com/content/datasheet/asset/file/PYU-RC_GROUP_51_ROHS_L"
 			(at 58.42 110.744 0)
 			(do_not_autoplace yes)
@@
 			)
 		)
-		(property "Link" ""
+		(property "Link" "https://yageogroup.com/products/Resistors/part/RC0402FR-071ML"
 			(at 58.674 112.268 0)
 			(do_not_autoplace yes)
@@
 			)
 		)
-		(property "MPN" ""
+		(property "MPN" "RC0402FR-071ML"
 			(at 58.42 114.3 0)
 			(do_not_autoplace yes)
@@
 			)
 		)
-		(property "MFG" ""
+		(property "MFG" "YAGEO"
 			(at 72.39 114.046 0)
 			(do_not_autoplace yes)
@@
 			)
 		)
-		(property "Datasheet" "url-ds"
+		(property "Datasheet" "https://app.adam-tech.com/products/download/data_sheet/201605/ph1-xx-ua-data-sheet.pdf"
 			(at 157.48 60.706 0)
 			(do_not_autoplace yes)
@@
 			)
 		)
-		(property "MPN" "MPN"
+		(property "MPN" "PH1-03-UA"
 			(at 157.48 54.864 0)
 			(do_not_autoplace yes)
@@
 			)
 		)
-		(property "MFG" "MFG"
+		(property "MFG" "Adam Tech"
 			(at 150.876 54.864 0)
 			(do_not_autoplace yes)
@@
 			)
 		)
-		(property "Link" "url-link"
+		(property "Link" ""
 			(at 157.48 59.436 0)
 			(do_not_autoplace yes)
@@
 			)
 		)
-		(property "Datasheet" ""
+		(property "Datasheet" "https://yageogroup.com/content/datasheet/asset/file/PYU-RC_GROUP_51_ROHS_L"
 			(at 80.01 41.656 0)
 			(do_not_autoplace yes)
@@
 			)
 		)
-		(property "Link" ""
+		(property "Link" "https://yageogroup.com/products/Resistors/part/RC0402FR-131KL"
 			(at 79.756 40.132 0)
 			(do_not_autoplace yes)
@@
 			)
 		)
-		(property "MPN" ""
+		(property "MPN" "RC0402FR-131KL"
 			(at 80.01 38.1 0)
 			(do_not_autoplace yes)
@@
 			)
 		)
-		(property "MFG" ""
+		(property "MFG" "YAGEO"
 			(at 66.04 38.354 0)
 			(do_not_autoplace yes)
@@
 			)
 		)
-		(property "Datasheet" ""
+		(property "Datasheet" "https://yageogroup.com/content/datasheet/asset/file/PYU-RC_GROUP_51_ROHS_L"
 			(at 112.014 146.05 0)
 			(do_not_autoplace yes)
@@
 			)
 		)
-		(property "MPN" ""
+		(property "MPN" "RC0402FR-0749R9L"
 			(at 115.57 146.05 0)
 			(do_not_autoplace yes)
@@
 			)
 		)
-		(property "MFG" ""
+		(property "MFG" "YAGEO"
 			(at 115.316 132.08 0)
 			(do_not_autoplace yes)
@@
 			)
 		)
-		(property "Link" ""
+		(property "Link" "https://yageogroup.com/products/Resistors/part/RC0402FR-0749R9L"
 			(at 115.57 102.235 0)
 			(do_not_autoplace yes)
@@
 			)
 		)
-		(property "Datasheet" ""
+		(property "Datasheet" "https://app.adam-tech.com/products/download/data_sheet/201605/ph1-xx-ua-data-sheet.pdf"
 			(at 58.42 137.414 0)
 			(do_not_autoplace yes)
@@
 			)
 		)
-		(property "MPN" ""
+		(property "MPN" "PH1-02-UA"
 			(at 58.42 143.256 0)
 			(do_not_autoplace yes)
@@
 			)
 		)
-		(property "MFG" ""
+		(property "MFG" "Adam Tech"
 			(at 51.816 143.256 0)
 			(do_not_autoplace yes)
@@
 			)
 		)
-		(property "Datasheet" ""
+		(property "Datasheet" "https://yageogroup.com/content/datasheet/asset/file/PYU-RC_GROUP_51_ROHS_L"
 			(at 111.76 36.576 0)
 			(do_not_autoplace yes)
@@
 			)
 		)
-		(property "Link" ""
+		(property "Link" "https://yageogroup.com/products/Resistors/part/RC0402FR-131KL"
 			(at 111.506 35.052 0)
 			(do_not_autoplace yes)
@@
 			)
 		)
-		(property "MPN" ""
+		(property "MPN" "RC0402FR-131KL"
 			(at 111.76 33.02 0)
 			(do_not_autoplace yes)
@@
 			)
 		)
-		(property "MFG" ""
+		(property "MFG" "YAGEO"
 			(at 97.79 33.274 0)
 			(do_not_autoplace yes)
@@
 			)
 		)
-		(property "Datasheet" ""
+		(property "Datasheet" "https://app.adam-tech.com/products/download/data_sheet/201605/ph1-xx-ua-data-sheet.pdf"
 			(at 100.076 92.71 0)
 			(do_not_autoplace yes)
@@
 			)
 		)
-		(property "MPN" ""
+		(property "MPN" "PH1-02-UA"
 			(at 94.234 92.71 0)
 			(do_not_autoplace yes)
@@
 			)
 		)
-		(property "MFG" ""
+		(property "MFG" "Adam Tech"
 			(at 94.234 86.106 0)
 			(do_not_autoplace yes)
@@
 			)
 		)
-		(property "Datasheet" ""
+		(property "Datasheet" "https://yageogroup.com/content/datasheet/asset/file/PYU-RC_GROUP_51_ROHS_L"
 			(at 96.52 71.374 0)
 			(do_not_autoplace yes)
@@
 			)
 		)
-		(property "Link" ""
+		(property "Link" "https://yageogroup.com/products/Resistors/part/RC0402FR-131KL"
 			(at 96.774 72.898 0)
 			(do_not_autoplace yes)
@@
 			)
 		)
-		(property "MPN" ""
+		(property "MPN" "RC0402FR-131KL"
 			(at 96.52 74.93 0)
 			(do_not_autoplace yes)
@@
 			)
 		)
-		(property "MFG" ""
+		(property "MFG" "YAGEO"
 			(at 110.49 74.676 0)
 			(do_not_autoplace yes)
