File: hw/pandore/pandore-rtmcu.kicad_sch (KiCad schematic)
At the start: 14 parts, among them J15 AIO, J16 DIO

Commit message: finished adding mpn,mfg to all parts, finished routing placement
Parts:
- JMP14: MFG (none) -> Adam Tech; MPN (none) -> PH1-02-UA
- R243, R244: Link (none) -> https://yageogroup.com/products/Resistors/part/RC0402FR-131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; MFG (none) -> YAGEO; MPN (none) -> RC0402FR-131KL
Connections:
- net VRTIO renamed V3P3
Other:
- note removed: "TODO: RTIO Voltage choice: 3.3V"
Changed lines of the file:
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@@
 		)
 	)
-	(text "TODO: RTIO Voltage choice: 3.3V"
-		(exclude_from_sim no)
-		(at 243.586 82.55 0)
-		(effects
-			(font
-				(size 1.016 1.016)
-			)
-		)
-	)
 	(text "SPI0.~{CS} / UART1.RX / I2C0.SCL / PWM2.B / CLOCK.GPOUT0"
 		(exclude_from_sim no)
@@
 	)
 	(junction
+		(at 60.96 24.13)
+		(diameter 0)
+		(color 0 0 0 0)
+	)
+	(junction
 		(at 254 104.14)
 		(diameter 0)
@@
 	(wire
 		(pts
-			(xy 60.96 43.18) (xy 60.96 45.72)
+			(xy 60.96 21.59) (xy 60.96 24.13)
 		)
 		(stroke
@@
 		)
 	)
+	(wire
+		(pts
+			(xy 60.96 24.13) (xy 73.66 24.13)
+		)
+		(stroke
+			(width 0)
+			(type default)
+		)
+	)
 	(bus
 		(pts
@@
 		)
 	)
-	(wire
-		(pts
-			(xy 64.77 24.13) (xy 73.66 24.13)
-		)
-		(stroke
-			(width 0)
-			(type default)
-		)
-	)
 	(bus
 		(pts
@@
 		)
 	)
+	(wire
+		(pts
+			(xy 60.96 24.13) (xy 60.96 45.72)
+		)
+		(stroke
+			(width 0)
+			(type default)
+		)
+	)
 	(bus
 		(pts
@@
 			)
 		)
-		(property "Datasheet" ""
+		(property "Datasheet" "https://app.adam-tech.com/products/download/data_sheet/201605/ph1-xx-ua-data-sheet.pdf"
 			(at 58.166 73.66 0)
 			(do_not_autoplace yes)
@@
 			)
 		)
-		(property "MPN" ""
+		(property "MPN" "PH1-02-UA"
 			(at 52.324 73.66 0)
 			(do_not_autoplace yes)
@@
 			)
 		)
-		(property "MFG" ""
+		(property "MFG" "Adam Tech"
 			(at 52.324 67.056 0)
 			(do_not_autoplace yes)
@@
 			)
 		)
-		(property "Datasheet" ""
+		(property "Datasheet" "https://yageogroup.com/content/datasheet/asset/file/PYU-RC_GROUP_51_ROHS_L"
 			(at 70.104 81.28 0)
 			(do_not_autoplace yes)
@@
 			)
 		)
-		(property "Link" ""
+		(property "Link" "https://yageogroup.com/products/Resistors/part/RC0402FR-131KL"
 			(at 71.628 81.026 0)
 			(do_not_autoplace yes)
@@
 			)
 		)
-		(property "MPN" ""
+		(property "MPN" "RC0402FR-131KL"
 			(at 73.66 81.28 0)
 			(do_not_autoplace yes)
@@
 			)
 		)
-		(property "MFG" ""
+		(property "MFG" "YAGEO"
 			(at 73.406 67.31 0)
 			(do_not_autoplace yes)
@@
 	)
 	(symbol
+		(lib_id "reekilib_pwr:VDD")
+		(at 60.96 20.32 0)
+		(unit 1)
+		(exclude_from_sim no)
+		(in_bom no)
+		(on_board no)
+		(dnp no)
+		(property "Reference" "#PWR0103"
+			(at 60.96 17.145 0)
+			(do_not_autoplace yes)
+			(effects
+				(font
+					(size 1 1)
+				)
+				(hide yes)
+			)
+		)
+		(property "Value" "V3P3"
+			(at 60.96 19.05 0)
+			(effects
+				(font
+					(size 1 1)
+				)
+			)
+		)
+		(property "Footprint" ""
+			(at 60.96 20.32 0)
+			(effects
+				(font
+					(size 1.524 1.524)
+				)
+			)
+		)
+		(property "Datasheet" ""
+			(at 60.96 20.32 0)
+			(effects
+				(font
+					(size 1.524 1.524)
+				)
+			)
+		)
+		(property "Description" ""
+			(at 60.96 20.32 0)
+			(effects
+				(font
+					(size 1.27 1.27)
+				)
+				(hide yes)
+			)
+		)
+		(pin "1"
+		)
+		(instances
+			(project "pandore"
+				(path "/e55f2700-f75a-4062-8a27-fe258faa8966/f774142b-755f-468a-93e0-eecae9257f8f"
+					(reference "#PWR0103")
+					(unit 1)
+				)
+			)
+		)
+	)
+	(symbol
 		(lib_id "reekilib_res:res_4")
 		(at 175.26 127 90)
@@
 			)
 		)
-		(property "Datasheet" ""
+		(property "Datasheet" "https://yageogroup.com/content/datasheet/asset/file/PYU-RC_GROUP_51_ROHS_L"
 			(at 67.564 66.04 0)
 			(do_not_autoplace yes)
@@
 			)
 		)
-		(property "Link" ""
+		(property "Link" "https://yageogroup.com/products/Resistors/part/RC0402FR-131KL"
 			(at 69.088 65.786 0)
 			(do_not_autoplace yes)
@@
 			)
 		)
-		(property "MPN" ""
+		(property "MPN" "RC0402FR-131KL"
 			(at 71.12 66.04 0)
 			(do_not_autoplace yes)
@@
 			)
 		)
-		(property "MFG" ""
+		(property "MFG" "YAGEO"
 			(at 70.866 52.07 0)
 			(do_not_autoplace yes)
