File: hw/pandore/pandore.kicad_sch (KiCad schematic)
At the start: 21 parts

Commit message: added monitor amp with volume knob continue routing all around
Other:
- sheet Computer ports: added PWRON; removed none
- sheet Power ports: added PWRON; removed none
Changed lines of the file:
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@@
 	(wire
 		(pts
+			(xy 76.2 35.56) (xy 118.11 35.56)
+		)
+		(stroke
+			(width 0)
+			(type default)
+		)
+	)
+	(wire
+		(pts
 			(xy 255.27 34.29) (xy 259.08 34.29)
 		)
@@
 			)
 		)
+		(pin "PWRON" input
+			(at 76.2 35.56 0)
+			(effects
+				(font
+					(size 1.016 1.016)
+				)
+				(justify right)
+			)
+		)
 		(instances
 			(project "pandore"
@@
 			(effects
 				(font
+					(size 1.016 1.016)
+				)
+				(justify left)
+			)
+		)
+		(pin "PWRON" output
+			(at 118.11 35.56 180)
+			(effects
+				(font

Commit message: last sprint almost done, most routing done
Other:
- sheet Computer ports: added none; removed SUSCLK
- sheet M.2 ports: added none; removed SUSCLK
Changed lines of the file:
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@@
 	(wire
 		(pts
-			(xy 76.2 35.56) (xy 118.11 35.56)
-		)
-		(stroke
-			(width 0)
-			(type default)
-		)
-	)
-	(wire
-		(pts
 			(xy 255.27 34.29) (xy 259.08 34.29)
 		)
@@
 	(wire
 		(pts
-			(xy 255.27 26.67) (xy 255.27 27.94)
+			(xy 76.2 35.56) (xy 118.11 35.56)
 		)
 		(stroke
@@
 	(wire
 		(pts
-			(xy 76.2 147.32) (xy 118.11 147.32)
+			(xy 255.27 26.67) (xy 255.27 27.94)
 		)
 		(stroke
@@
 		)
 	)
-	(bus
+	(wire
 		(pts
-			(xy 76.2 142.24) (xy 118.11 142.24)
+			(xy 76.2 147.32) (xy 118.11 147.32)
 		)
 		(stroke
@@
 	(bus
 		(pts
-			(xy 177.8 34.29) (xy 200.66 34.29)
+			(xy 76.2 142.24) (xy 118.11 142.24)
 		)
 		(stroke
@@
 		)
 	)
-	(wire
+	(bus
 		(pts
-			(xy 262.89 20.32) (xy 266.7 20.32)
+			(xy 177.8 34.29) (xy 200.66 34.29)
 		)
 		(stroke
@@
 	(wire
 		(pts
-			(xy 76.2 49.53) (xy 118.11 49.53)
+			(xy 262.89 20.32) (xy 266.7 20.32)
 		)
 		(stroke
@@
 			)
 		)
-		(pin "SUSCLK" output
-			(at 118.11 49.53 180)
-			(effects
-				(font
-					(size 1.016 1.016)
-				)
-				(justify left)
-			)
-		)
 		(pin "MGMTMCU{USB2}" bidirectional
 			(at 118.11 88.9 180)
@@
 			(effects
 				(font
-					(size 1.016 1.016)
-				)
-				(justify right)
-			)
-		)
-		(pin "SUSCLK" input
-			(at 76.2 49.53 0)
-			(effects
-				(font

Commit message: all routed, review starting
Other:
- sheet Audio ports: added EN; removed none
- sheet Computer ports: added AUDIO.EN, VUSB.EN; removed none
- sheet USB ports ports: added VUSB.EN; removed none
Changed lines of the file:
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@@
 		)
 	)
+	(wire
+		(pts
+			(xy 177.8 60.96) (xy 200.66 60.96)
+		)
+		(stroke
+			(width 0)
+			(type default)
+		)
+	)
 	(bus
 		(pts
@@
 		)
 	)
+	(wire
+		(pts
+			(xy 76.2 130.81) (xy 118.11 130.81)
+		)
+		(stroke
+			(width 0)
+			(type default)
+		)
+	)
 	(bus
 		(pts
@@
 			)
 		)
+		(pin "VUSB.EN" output
+			(at 177.8 60.96 0)
+			(effects
+				(font
+					(size 1.016 1.016)
+				)
+				(justify right)
+			)
+		)
+		(pin "AUDIO.EN" output
+			(at 118.11 130.81 180)
+			(effects
+				(font
+					(size 1.016 1.016)
+				)
+				(justify left)
+			)
+		)
 		(instances
 			(project "pandore"
@@
 	)
 	(sheet
-		(at 33.02 133.35)
-		(size 43.18 19.05)
+		(at 33.02 128.27)
+		(size 43.18 24.13)
 		(exclude_from_sim no)
 		(in_bom yes)
@@
 		)
 		(property "Sheetname" "Audio"
-			(at 53.975 137.16 0)
+			(at 53.975 132.08 0)
 			(do_not_autoplace yes)
 			(effects
@@
 		)
 		(property "Sheetfile" "pandore-audio.kicad_sch"
-			(at 33.528 170.942 0)
+			(at 33.528 165.862 0)
 			(effects
 				(font
@@
 		)
 		(property "pageNb" "Page ${#}"
-			(at 53.975 140.97 0)
+			(at 53.975 135.89 0)
 			(effects
 				(font
@@
 			)
 		)
+		(pin "EN" input
+			(at 76.2 130.81 0)
+			(effects
+				(font
+					(size 1.016 1.016)
+				)
+				(justify right)
+			)
+		)
 		(instances
 			(project "pandore"
@@
 	(sheet
 		(at 200.66 39.37)
-		(size 43.18 21.59)
+		(size 43.18 24.13)
 		(exclude_from_sim no)
 		(in_bom yes)
@@
 			)
 		)
+		(pin "VUSB.EN" input
+			(at 200.66 60.96 180)
+			(effects
+				(font
+					(size 1.016 1.016)
+				)
+				(justify left)
+			)
+		)
 		(instances
 			(project "pandore"
@@
 	)
 	(sheet
-		(at 200.66 62.23)
-		(size 43.18 16.51)
+		(at 200.66 64.77)
+		(size 43.18 13.97)
 		(exclude_from_sim no)
 		(in_bom yes)
@@
 		)
 		(property "Sheetname" "Display"
-			(at 221.615 66.04 0)
+			(at 221.615 68.58 0)
 			(do_not_autoplace yes)
 			(effects
@@
 		)
 		(property "Sheetfile" "pandore-display.kicad_sch"
-			(at 201.168 99.822 0)
+			(at 201.168 102.362 0)
 			(effects
 				(font
@@
 		)
 		(property "pageNb" "Page ${#}"
-			(at 221.615 69.85 0)
+			(at 221.615 72.39 0)
 			(effects
 				(font

Commit message: finished adding mpn,mfg to all parts, finished routing placement
Parts:
- C1, R1: now not fitted
Other:
- sheet Display ports: added DISABLE; removed none
Changed lines of the file:
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@@
 		(length 1.27)
 		(shape diamond)
-		(at 83.82 25.4 180)
-		(fields_autoplaced yes)
-		(effects
-			(font
-				(size 1.016 1.016)
-			)
-			(justify right bottom)
-		)
-		(property "Netclass" "PWR"
-			(at 84.9173 26.67 0)
-			(effects
-				(font
-					(size 1.27 1.27)
-				)
-				(justify left)
-			)
-		)
-		(property "Component Class" ""
-			(at -87.63 -73.66 0)
-			(effects
-				(font
-					(size 1.27 1.27)
-					(italic yes)
-				)
-			)
-		)
-	)
-	(netclass_flag ""
-		(length 1.27)
-		(shape diamond)
 		(at 83.82 30.48 0)
 		(fields_autoplaced yes)
@@
 		(in_bom yes)
 		(on_board yes)
-		(dnp no)
+		(dnp yes)
 		(property "Reference" "C1"
 			(at 252.73 27.686 0)
@@
 		(in_bom yes)
 		(on_board yes)
-		(dnp no)
+		(dnp yes)
 		(property "Reference" "R1"
 			(at 261.112 27.686 0)
@@
 	)
 	(symbol
-		(lib_id "reekilib_pwr:VDD")
-		(at 83.82 24.13 0)
-		(unit 1)
-		(exclude_from_sim no)
-		(in_bom no)
-		(on_board no)
-		(dnp no)
-		(property "Reference" "#PWR01"
-			(at 83.82 20.955 0)
-			(do_not_autoplace yes)
-			(effects
-				(font
-					(size 1 1)
-				)
-				(hide yes)
-			)
-		)
-		(property "Value" "VDD"
-			(at 83.82 23.114 0)
-			(effects
-				(font
-					(size 1 1)
-				)
-			)
-		)
-		(property "Footprint" ""
-			(at 83.82 24.13 0)
-			(effects
-				(font
-					(size 1.524 1.524)
-				)
-			)
-		)
-		(property "Datasheet" ""
-			(at 83.82 24.13 0)
-			(effects
-				(font
-					(size 1.524 1.524)
-				)
-			)
-		)
-		(property "Description" ""
-			(at 83.82 24.13 0)
-			(effects
-				(font
-					(size 1.27 1.27)
-				)
-				(hide yes)
-			)
-		)
-		(pin "1"
-		)
-		(instances
-			(project ""
-				(path "/e55f2700-f75a-4062-8a27-fe258faa8966"
-					(reference "#PWR01")
-					(unit 1)
-				)
-			)
-		)
-	)
-	(symbol
 		(lib_id "reekilib_vrt:virtual")
 		(at 238.76 143.51 0)
@@
 			(effects
 				(font
+					(size 1.016 1.016)
+				)
+				(justify left)
+			)
+		)
+		(pin "DISABLE" input
+			(at 200.66 74.93 180)
+			(effects
+				(font
